File: d69-80.kicad_pcb (KiCad board)
At the start: 2 copper layers, 163 parts, among them SW1 SW_Push, SW10 SW_Push, SW101 SW_SPST, SW11 SW_Push, SW12 SW_Push, SW13 SW_Push, SW14 SW_Push, SW15 SW_Push, SW16 SW_Push, SW17 SW_Push, SW18 SW_Push, SW19 SW_Push, SW2 SW_Push, SW20 SW_Push, SW21 SW_Push, SW22 SW_Push, SW23 SW_Push, SW24 SW_Push, SW25 SW_Push, SW26 SW_Push, SW27 SW_Push, SW28 SW_Push, SW29 SW_Push, SW3 SW_Push, SW30 SW_Push, SW31 SW_Push, SW32 SW_Push, SW33 SW_Push, SW34 SW_Push, SW35 SW_Push, SW36 SW_Push, SW37 SW_Push, SW38 SW_Push, SW39 SW_Push, SW4 SW_Push, SW40 SW_Push, SW41 SW_Push, SW42 SW_Push, SW43 SW_Push, SW44 SW_Push, SW45 SW_Push, SW46 SW_Push, SW47 SW_Push, SW48 SW_Push, SW49 SW_Push, SW5 SW_Push, SW50 SW_Push, SW51 SW_Push, SW52 SW_Push, SW53 SW_Push, SW54 SW_Push, SW55 SW_Push, SW56 SW_Push, SW57 SW_Push, SW58 SW_Push, SW59 SW_Push, SW6 SW_Push, SW60 SW_Push, SW61 SW_Push, SW62 SW_Push, SW63 SW_Push, SW64 SW_Push, SW65 SW_Push, SW66 SW_Push, SW67 SW_Push, SW68 SW_Push, SW69 SW_Push, SW7 SW_Push, SW70 SW_Push, SW71 SW_Push, SW72 SW_Push, SW73 SW_Push, SW74 SW_Push, SW75 SW_Push, SW76 SW_Push, SW77 SW_Push, SW78 SW_Push, SW79 SW_Push, SW8 SW_Push, SW80 SW_Push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

Commit message: adds mcu and io-expander, initial wiring
Parts:
- added U1: xiao-ble, Library:xiao-ble-smd-cutout, B.Cu at (36.3, 45.8)
- added U2: ~, Library:QFN-32_EP_5x5_Pitch0.5mm, B.Cu at (135.0, 119.0)
- moved D1 4.17 mm to (48.5, 38.2)
- moved D15 4.17 mm to (48.5, 55.2)
- moved D29 4.17 mm to (50.8, 72.2)
Routing:
- net /SDA: track 0.00 -> 187.6 mm, vias 0 -> 1
- net /VCC: track 0.00 -> 182.8 mm, vias 0 -> 3
- net /GND: track 0.00 -> 181.2 mm, vias 0 -> 2
- net /SCL: track 0.00 -> 179.2 mm, vias 0 -> 1
- net /COL13: track 92.5 -> 238.3 mm, vias 0 -> 2
- net /COL12: track 96.2 -> 222.7 mm, vias 0 -> 2
- net /COL11: track 96.2 -> 202.6 mm, vias 0 -> 2
- net /COL00: track 88.7 -> 193.8 mm, vias 0 -> 2
- net /COL01: track 92.5 -> 181.5 mm, vias 0 -> 2
- net /COL10: track 96.2 -> 182.7 mm, vias 0 -> 2
- net /ROW0: track 269.9 -> 354.4 mm, vias 14 -> 16
- net /COL02: track 92.5 -> 164.8 mm, vias 0 -> 2
- net /COL09: track 96.2 -> 166.1 mm, vias 0 -> 2
- net /ROW1: track 266.7 -> 326.5 mm, vias 14 -> 15
- net /COL03: track 92.5 -> 147.5 mm, vias 0 -> 2
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Other:
- board outline added: 8.8 x 6.2 mm

Commit message: adds leds, connects switch and some cleanup
Parts:
- added D82: LED, LED_SMD:LED_0603_1608Metric_Pad1.05x0.95mm_HandSolder, F.Cu at (54.0, 39.4)
- added D83: LED, LED_SMD:LED_0603_1608Metric_Pad1.05x0.95mm_HandSolder, F.Cu at (72.0, 39.4)
- added D84: LED, LED_SMD:LED_0603_1608Metric_Pad1.05x0.95mm_HandSolder, F.Cu at (90.0, 39.4)
- added J1: Conn_01x02_Socket, Connector_JST:JST_XH_B2B-XH-AM_1x02_P2.50mm_Vertical, B.Cu at (109.2, 38.6)
- added R1: R, Resistor_SMD:R_0603_1608Metric_Pad0.98x0.95mm_HandSolder, F.Cu at (90.0, 38.0)
- added R2: R, Resistor_SMD:R_0603_1608Metric_Pad0.98x0.95mm_HandSolder, F.Cu at (72.0, 38.0)
- added R3: R, Resistor_SMD:R_0603_1608Metric_Pad0.98x0.95mm_HandSolder, F.Cu at (54.0, 38.0)
Connections:
- SW101 pad 1: unconnected-(SW101-A-Pad1) -> /BATSW
- SW101 pad 2: unconnected-(SW101-B-Pad2) -> /BAT+
- U1 pad 10: unconnected-(U1-A5_MISO/1.14-Pad10) -> /LED1
- U1 pad 19: unconnected-(U1-BAT-Pad19) -> /BATSW
- U1 pad 8: unconnected-(U1-B9_RX/1.12-Pad8) -> /LED2
- U1 pad 9: unconnected-(U1-A7_SCK/1.13-Pad9) -> /LED0
- U2 pad 33: (no net) -> /GND
Routing:
- net /BATSW: track 0.00 -> 337.8 mm, vias 0 -> 1
- net /BAT+: track 0.00 -> 251.8 mm
- net /GND: track 181.2 -> 318.0 mm, vias 2 -> 3
- net /LED2: track 0.00 -> 55.0 mm
- net /LED1: track 0.00 -> 44.1 mm
- net /LED0: track 0.00 -> 21.0 mm
- net /ROW0: track 354.4 -> 362.4 mm, vias 16 -> 15
- net /SDA: track 187.6 -> 182.2 mm, vias 1 -> 2
- net /ROW2: track 314.3 -> 310.7 mm
- net /ROW3: track 275.7 -> 272.6 mm
- net /COL00: track 193.8 -> 195.9 mm
- net /COL09: track 166.1 -> 164.0 mm
- net /ROW4: track 276.7 -> 275.1 mm
- net Net-(D82-K): track 0.00 -> 1.44 mm
- net Net-(D84-K): track 0.00 -> 1.42 mm
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Other:
- board outline removed

Commit message: more cleanup
Parts:
- moved SW101 8.45 mm to (276.1, 119.4)
- moved D10 8.45 mm to (207.1, 36.1)
- moved D11 8.45 mm to (225.1, 36.1)
- moved D12 8.45 mm to (243.1, 36.1)
- moved D17 8.45 mm to (72.1, 53.1)
- moved D18 8.45 mm to (90.1, 53.1)
- moved D19 8.45 mm to (108.1, 53.1)
- moved D20 8.45 mm to (126.1, 53.1)
- moved D21 8.45 mm to (144.1, 53.1)
- moved D22 8.45 mm to (162.1, 53.1)
- moved D23 8.45 mm to (180.1, 53.1)
- moved D24 8.45 mm to (198.1, 53.1)
- moved D25 8.45 mm to (216.1, 53.1)
- moved D26 8.45 mm to (234.1, 53.1)
- moved D27 8.45 mm to (252.1, 53.1)
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Routing:
- net /ROW1: track 326.5 -> 320.4 mm
- net /ROW0: track 362.4 -> 356.8 mm, vias 15 -> 14
- net /SDA: track 182.2 -> 187.2 mm
- net /COL06: track 112.8 -> 117.5 mm
- net /ROW4: track 275.1 -> 270.5 mm
- net /ROW2: track 310.7 -> 306.5 mm, vias 15 -> 14
- net /COL03: track 147.4 -> 151.6 mm
- net /SCL: track 180.0 -> 184.0 mm
- net /COL04: track 123.2 -> 126.5 mm
- net /COL11: track 202.6 -> 205.6 mm
- net /COL07: track 116.8 -> 119.8 mm
- net /COL10: track 182.6 -> 185.6 mm
- net /COL12: track 222.4 -> 225.3 mm
- net /COL09: track 164.0 -> 166.7 mm
- net /COL01: track 181.2 -> 183.8 mm
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
Commit message: even more cleanup.. still wip
Routing:
- net /ROW3: track 273.3 -> 263.5 mm
- net /ROW2: track 306.5 -> 301.0 mm, vias 14 -> 15
- net /COL12: track 225.3 -> 228.3 mm
- net /COL11: track 205.6 -> 208.6 mm
- net /COL10: track 185.6 -> 188.6 mm
- net /COL09: track 166.7 -> 169.7 mm
- net /COL08: track 137.3 -> 140.3 mm
- net /ROW1: track 320.4 -> 317.8 mm
- net /COL04: track 126.5 -> 129.0 mm
- net /COL02: track 167.4 -> 169.7 mm
- net /COL01: track 183.8 -> 186.1 mm
- net /ROW4: track 270.5 -> 268.4 mm
- net /COL03: track 151.6 -> 153.3 mm
- net /ROW0: track 356.8 -> 358.4 mm
- net /BAT+: track 252.6 -> 251.1 mm
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
Commit message: Add I2C pullups (oops), switch to wakeup switch from battery cutoff
Parts:
- added R4: R, Resistor_SMD:R_0603_1608Metric_Pad0.98x0.95mm_HandSolder, B.Cu at (121.6, 114.2)
- added R5: R, Resistor_SMD:R_0603_1608Metric_Pad0.98x0.95mm_HandSolder, B.Cu at (121.0, 115.8)
- SW101: footprint Button_Switch_SMD:SW_DIP_SPSTx01_Slide_9.78x4.72mm_W8.61mm_P2.54mm -> Library:combo
- moved SW101 1.59 mm to (275.1, 118.1)
- moved R1 0.20 mm to (81.6, 37.3)
- moved R2 0.20 mm to (63.6, 37.3)
- moved R3 0.20 mm to (45.6, 37.3)
- moved D82 0.20 mm to (45.6, 38.7)
- moved D83 0.20 mm to (63.6, 38.7)
- moved D84 0.20 mm to (81.6, 38.7)
Connections:
- SW101 pad 1: /BATSW -> /GND
- SW101 pad 2: /BAT+ -> /BOOT
- U1 pad 19: /BATSW -> /BAT+
- U1 pad 7: unconnected-(U1-B8_TX/1.11-Pad7) -> /BOOT
Routing:
- net /BATSW: track 335.9 -> 0.00 mm, vias 1 -> 0
- net /BOOT: track 0.00 -> 326.9 mm
- net /GND: track 317.8 -> 582.6 mm
- net /BAT+: track 251.1 -> 76.6 mm, vias 0 -> 1
- net /SDA: track 186.0 -> 191.3 mm, vias 2 -> 3
- net /SCL: track 183.5 -> 188.1 mm, vias 2 -> 3
- net /VCC: track 180.7 -> 185.2 mm
- net /ROW0: track 358.4 -> 359.7 mm
- net /LED2: track 55.2 -> 56.2 mm
